File: schematics/register_file/register_file.kicad_sch (KiCad schematic)
At the start: 30 parts, among them J1 Conn_02x25_Counter_Clockwise, U1 74LS08, U2 74LS574, U3 74HC04, U4 74HC04, U5 74HC04, U6 74LS08, U7 74LS32, U8 74LS08

Commit message: fixed all errors
Parts:
- removed U4, U5: 74HC04, symbol 74xx:74HC04
- removed U6, U8: 74LS08, symbol 74xx:74LS08
- removed U7: 74LS32, symbol 74xx:74LS32
- added unit 5 of U1
- added unit 1 of U1
- added unit 4 of U1
- added unit 2 of U1
- added unit 2 of U3
- added unit 3 of U3
- added unit 7 of U3
- added U4: 74LS08, Package_DIP:DIP-14_W7.62mm_Socket_LongPads, symbol 74xx:74LS08
- added U5: 74LS32, symbol 74xx:74LS32
- U1, U3: footprint (none) -> Package_DIP:DIP-14_W7.62mm_Socket_LongPads
- renumbered ALU_BUFFER_IN to B_IN0, DBUS_BUFFER_IN to B_IN1, BUFFER_OUT to B_OUT0
Connections:
- net ALU0: now also B_IN0.11 (B7); no longer B_IN0.2 (A0), B_IN0.9 (A7), J1.17 (Pin_17)
- net ALU1: now also B_IN0.12 (B6); no longer B_IN0.3 (A1), B_IN0.8 (A6), J1.16 (Pin_16)
- net ALU2: now also B_IN0.13 (B5); no longer B_IN0.4 (A2), B_IN0.7 (A5), J1.15 (Pin_15)
- net GND: now also B_IN0.1 (A->B), B_IN0.14 (B4), B_IN0.15 (B3), B_IN0.16 (B2), B_IN0.17 (B1), B_IN0.18 (B0), B_IN1.1 (A->B), B_OUT0.1 (A->B), R5.2, R6.2, U2.1 (OE), U1.7 (GND), U3.7 (GND), U4.14 (VCC), U5.7 (GND)
- net LOAD_FR: now also U5.2
- net LOAD_R0: now also U1.12
- net LOAD_R1: now also U4.1
- net LOAD_R2: now also U1.1; no longer U1.9
- net LOAD_R3: now also U1.4
- net LOAD_R4: now also U4.4
- net OUT_FR: now also U3.5
- net UPDATE_FR: now also U3.3, U5.1
- net VCC: now also B_IN1.11 (B7), B_IN1.12 (B6), B_IN1.13 (B5), B_IN1.14 (B4), B_IN1.15 (B3), B_IN1.16 (B2), B_IN1.17 (B1), B_IN1.18 (B0), B_OUT0.2 (A0), B_OUT0.3 (A1), B_OUT0.4 (A2), B_OUT0.5 (A3), B_OUT0.6 (A4), B_OUT0.7 (A5), B_OUT0.8 (A6), B_OUT0.9 (A7), J1.1 (Pin_1), J1.2 (Pin_2), J1.3 (Pin_3), J1.4 (Pin_4), J1.5 (Pin_5), J1.6 (Pin_6), J1.7 (Pin_7), J1.8 (Pin_8), R0.12 (Q7), R0.13 (Q6), R0.14 (Q5), R0.15 (Q4), R0.16 (Q3), R0.17 (Q2), R0.18 (Q1), R0.19 (Q0), R0.2 (D0), R0.3 (D1), R0.4 (D2), R0.5 (D3), R0.6 (D4), R0.7 (D5), R0.8 (D6), R0.9 (D7), R1.12 (Q7), R1.13 (Q6), R1.14 (Q5), R1.15 (Q4), R1.16 (Q3), R1.17 (Q2), R1.18 (Q1), R1.19 (Q0), R1.2 (D0), R1.3 (D1), R1.4 (D2), R1.5 (D3), R1.6 (D4), R1.7 (D5), R1.8 (D6), R1.9 (D7), R2.12 (Q7), R2.13 (Q6), R2.14 (Q5), R2.15 (Q4), R2.16 (Q3), R2.17 (Q2), R2.18 (Q1), R2.19 (Q0), R2.2 (D0), R2.3 (D1), R2.4 (D2), R2.5 (D3), R2.6 (D4), R2.7 (D5), R2.8 (D6), R2.9 (D7), R3.12 (Q7), R3.13 (Q6), R3.14 (Q5), R3.15 (Q4), R3.16 (Q3), R3.17 (Q2), R3.18 (Q1), R3.19 (Q0), R3.2 (D0), R3.3 (D1), R3.4 (D2), R3.5 (D3), R3.6 (D4), R3.7 (D5), R3.8 (D6), R3.9 (D7), R4.12 (Q7), R4.13 (Q6), R4.14 (Q5), R4.15 (Q4), R4.16 (Q3), R4.17 (Q2), R4.18 (Q1), R4.19 (Q0), R4.2 (D0), R4.3 (D1), R4.4 (D2), R4.5 (D3), R4.6 (D4), R4.7 (D5), R4.8 (D6), R4.9 (D7), R5.1, R6.1, R7.1, R8.1, U1.14 (VCC), U3.14 (VCC), U4.7 (GND), U5.14 (VCC); no longer R5.2, R6.2
- net ~CLK: now also U1.9, U1.13, U1.2, U1.5, U4.2, U4.5; no longer U1.10
- net at U2.11 (Cp): now also U1.8
- net at R2.11 (Cp): now also U1.3; no longer U1.8
- net at R3.11 (Cp): now also U1.6
- net at B_IN0.19 (CE): now also U3.4
- net at B_OUT0.19 (CE): now also U3.6
- net at U2.12 (Q7): now also B_OUT0.11 (B7); no longer B_OUT0.9 (A7)
- net at U2.13 (Q6): now also B_OUT0.12 (B6); no longer B_OUT0.8 (A6)
- net at U2.14 (Q5): now also B_OUT0.13 (B5); no longer B_OUT0.7 (A5)
- net at U2.15 (Q4): now also B_OUT0.14 (B4); no longer B_OUT0.6 (A4)
- net at U2.16 (Q3): now also B_OUT0.15 (B3); no longer B_OUT0.5 (A3)
- net at U2.17 (Q2): now also B_OUT0.16 (B2); no longer B_OUT0.4 (A2)
- net at U2.18 (Q1): now also B_OUT0.17 (B1); no longer B_OUT0.3 (A1)
- net at U2.19 (Q0): now also B_OUT0.18 (B0); no longer B_OUT0.2 (A0)
- net at R0.11 (Cp): now also U1.11
- net at R4.11 (Cp): now also U4.6
- net at R1.11 (Cp): now also U4.3
- removed net ALU3: B_IN0.5 (A3), B_IN0.6 (A4), J1.13 (Pin_13), J1.14 (Pin_14)
- removed net D0: B_IN1.2 (A0), B_OUT0.18 (B0), J1.1 (Pin_1), R0.19 (Q0), R0.2 (D0), R1.19 (Q0), R1.2 (D0), R2.19 (Q0), R2.2 (D0), R3.19 (Q0), R3.2 (D0), R4.19 (Q0), R4.2 (D0)
- removed net D1: B_IN1.3 (A1), B_OUT0.17 (B1), J1.2 (Pin_2), R0.18 (Q1), R0.3 (D1), R1.18 (Q1), R1.3 (D1), R2.18 (Q1), R2.3 (D1), R3.18 (Q1), R3.3 (D1), R4.18 (Q1), R4.3 (D1)
- removed net D2: B_IN1.4 (A2), B_OUT0.16 (B2), J1.3 (Pin_3), R0.17 (Q2), R0.4 (D2), R1.17 (Q2), R1.4 (D2), R2.17 (Q2), R2.4 (D2), R3.17 (Q2), R3.4 (D2), R4.17 (Q2), R4.4 (D2)
- removed net D3: B_IN1.5 (A3), B_OUT0.15 (B3), J1.4 (Pin_4), R0.16 (Q3), R0.5 (D3), R1.16 (Q3), R1.5 (D3), R2.16 (Q3), R2.5 (D3), R3.16 (Q3), R3.5 (D3), R4.16 (Q3), R4.5 (D3)
- removed net D4: B_IN1.6 (A4), B_OUT0.14 (B4), J1.5 (Pin_5), R0.15 (Q4), R0.6 (D4), R1.15 (Q4), R1.6 (D4), R2.15 (Q4), R2.6 (D4), R3.15 (Q4), R3.6 (D4), R4.15 (Q4), R4.6 (D4)
- removed net D5: B_IN1.7 (A5), B_OUT0.13 (B5), J1.6 (Pin_6), R0.14 (Q5), R0.7 (D5), R1.14 (Q5), R1.7 (D5), R2.14 (Q5), R2.7 (D5), R3.14 (Q5), R3.7 (D5), R4.14 (Q5), R4.7 (D5)
- removed net D6: B_IN1.8 (A6), B_OUT0.12 (B6), J1.7 (Pin_7), R0.13 (Q6), R0.8 (D6), R1.13 (Q6), R1.8 (D6), R2.13 (Q6), R2.8 (D6), R3.13 (Q6), R3.8 (D6), R4.13 (Q6), R4.8 (D6)
- removed net D7: B_IN1.9 (A7), B_OUT0.11 (B7), J1.8 (Pin_8), R0.12 (Q7), R0.9 (D7), R1.12 (Q7), R1.9 (D7), R2.12 (Q7), R2.9 (D7), R3.12 (Q7), R3.9 (D7), R4.12 (Q7), R4.9 (D7)
- new net: U1.10, U5.3
- new net: B_IN1.2 (A0), U2.2 (D0)
- new net: B_IN1.3 (A1), U2.3 (D1)
- new net: B_IN1.4 (A2), U2.4 (D2)
- new net: B_IN1.5 (A3), U2.5 (D3)
- new net: B_IN1.6 (A4), U2.6 (D4)
- new net: B_IN0.7 (A5), B_IN1.7 (A5), U2.7 (D5)
- new net: B_IN0.8 (A6), B_IN1.8 (A6), U2.8 (D6)
- new net: B_IN0.9 (A7), B_IN1.9 (A7), U2.9 (D7)
- no-connect marks 18 -> 28
Other:
- moved on the sheet: B_IN0, B_IN1, B_OUT0, C1, C2, C3, C4, C5, C6, C8, C9, J1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

Commit message: Connnect all modules together
Parts:
- removed R5, R6, R7, R8: R, symbol Device:R
- removed U1, U4: 74LS08, Package_DIP:DIP-14_W7.62mm_Socket_LongPads, symbol 74xx:74LS08
- removed U3: 74HC04, Package_DIP:DIP-14_W7.62mm_Socket_LongPads, symbol 74xx:74HC04
- removed U5: 74LS32, symbol 74xx:74LS32
- added C10, C11, C12: C, symbol Device:C
- added U1, U3: 74LS02, symbol 74xx:74LS02
- added U4: 74LS04, symbol 74xx:74LS04
- J1: footprint (none) -> Connector_PinSocket_2.54mm:PinSocket_2x25_P2.54mm_Horizontal
- R0, R1, R2, R3, R4: footprint (none) -> Package_DIP:DIP-20_W7.62mm_Socket_LongPads
Connections:
- net OUT_FR is gone; now on net ~{OUT_FR}: J1.40 (Pin_40)
- net UPDATE_FR is gone; now on net ~{UPDATE_FR}: J1.28 (Pin_28)
- net GND: now also J1.10 (Pin_10), J1.19 (Pin_19), J1.2 (Pin_2), J1.49 (Pin_49), C10.2, C11.2, C12.2, U1.7 (GND), U3.7 (GND), U4.7 (GND); no longer J1.50 (Pin_50)
- net VCC: now also J1.25 (Pin_25), J1.26 (Pin_26), J1.50 (Pin_50), C10.1, C11.1, C12.1, U1.14 (VCC), U3.14 (VCC), U4.14 (VCC); no longer B_IN1.11 (B7), B_IN1.12 (B6), B_IN1.13 (B5), B_IN1.14 (B4), B_IN1.15 (B3), B_IN1.16 (B2), B_IN1.17 (B1), B_IN1.18 (B0), B_OUT0.2 (A0), B_OUT0.3 (A1), B_OUT0.4 (A2), B_OUT0.5 (A3), B_OUT0.6 (A4), B_OUT0.7 (A5), B_OUT0.8 (A6), B_OUT0.9 (A7), J1.2 (Pin_2), J1.3 (Pin_3), J1.4 (Pin_4), J1.49 (Pin_49), J1.5 (Pin_5), J1.6 (Pin_6), J1.7 (Pin_7), J1.8 (Pin_8), R0.12 (Q7), R0.13 (Q6), R0.14 (Q5), R0.15 (Q4), R0.16 (Q3), R0.17 (Q2), R0.18 (Q1), R0.19 (Q0), R0.2 (D0), R0.3 (D1), R0.4 (D2), R0.5 (D3), R0.6 (D4), R0.7 (D5), R0.8 (D6), R0.9 (D7), R1.12 (Q7), R1.13 (Q6), R1.14 (Q5), R1.15 (Q4), R1.16 (Q3), R1.17 (Q2), R1.18 (Q1), R1.19 (Q0), R1.2 (D0), R1.3 (D1), R1.4 (D2), R1.5 (D3), R1.6 (D4), R1.7 (D5), R1.8 (D6), R1.9 (D7), R2.12 (Q7), R2.13 (Q6), R2.14 (Q5), R2.15 (Q4), R2.16 (Q3), R2.17 (Q2), R2.18 (Q1), R2.19 (Q0), R2.2 (D0), R2.3 (D1), R2.4 (D2), R2.5 (D3), R2.6 (D4), R2.7 (D5), R2.8 (D6), R2.9 (D7), R3.12 (Q7), R3.13 (Q6), R3.14 (Q5), R3.15 (Q4), R3.16 (Q3), R3.17 (Q2), R3.18 (Q1), R3.19 (Q0), R3.2 (D0), R3.3 (D1), R3.4 (D2), R3.5 (D3), R3.6 (D4), R3.7 (D5), R3.8 (D6), R3.9 (D7), R4.12 (Q7), R4.13 (Q6), R4.14 (Q5), R4.15 (Q4), R4.16 (Q3), R4.17 (Q2), R4.18 (Q1), R4.19 (Q0), R4.2 (D0), R4.3 (D1), R4.4 (D2), R4.5 (D3), R4.6 (D4), R4.7 (D5), R4.8 (D6), R4.9 (D7)
- net ~CLK: now also J1.3 (Pin_3), U1.12, U1.3, U1.6, U1.9, U3.3, U3.8; no longer J1.26 (Pin_26)
- net at R2.11 (Cp): now also U1.10
- net ~{UPDATE_FR}: now reaches B_IN0.19 (CE)
- net ~{UPDATE_FR}: now also B_IN1.19 (CE), U4.5
- net at U2.11 (Cp): now also U3.10
- net ZeroOut: now reaches B_OUT0.11 (B7), U2.12 (Q7)
- net ZeroOut: now also J1.44 (Pin_44)
- net ~{CarryOut}: now reaches B_OUT0.12 (B6), U2.13 (Q6)
- net ~{CarryOut}: now also J1.45 (Pin_45)
- net SignOut: now reaches B_OUT0.13 (B5), U2.14 (Q5)
- net SignOut: now also J1.46 (Pin_46)
- net at B_IN1.2 (A0), U2.2 (D0): now also B_IN0.2 (A0)
- net at B_IN1.3 (A1), U2.3 (D1): now also B_IN0.3 (A1)
- net at B_IN1.4 (A2), U2.4 (D2): now also B_IN0.4 (A2)
- net at B_IN1.5 (A3), U2.5 (D3): now also B_IN0.5 (A3)
- net at B_IN1.6 (A4), U2.6 (D4): now also B_IN0.6 (A4)
- net ~{OUT_FR}: now reaches B_OUT0.19 (CE)
- net at R0.11 (Cp): now also U1.1
- net at R1.11 (Cp): now also U3.1
- net at R4.11 (Cp): now also U1.4
- net at R3.11 (Cp): now also U1.13
- net D2: now reaches J1.13 (Pin_13)
- net D2: now also B_IN1.16 (B2), B_OUT0.4 (A2), R0.17 (Q2), R0.4 (D2), R1.17 (Q2), R1.4 (D2), R2.17 (Q2), R2.4 (D2), R3.17 (Q2), R3.4 (D2), R4.17 (Q2), R4.4 (D2)
- net D3: now reaches J1.14 (Pin_14)
- net D3: now also B_IN1.15 (B3), B_OUT0.5 (A3), R0.16 (Q3), R0.5 (D3), R1.16 (Q3), R1.5 (D3), R2.16 (Q3), R2.5 (D3), R3.16 (Q3), R3.5 (D3), R4.16 (Q3), R4.5 (D3)
- net D4: now reaches J1.15 (Pin_15)
- net D4: now also B_IN1.14 (B4), B_OUT0.6 (A4), R0.15 (Q4), R0.6 (D4), R1.15 (Q4), R1.6 (D4), R2.15 (Q4), R2.6 (D4), R3.15 (Q4), R3.6 (D4), R4.15 (Q4), R4.6 (D4)
- net D5: now reaches J1.16 (Pin_16)
- net D5: now also B_IN1.13 (B5), B_OUT0.7 (A5), R0.14 (Q5), R0.7 (D5), R1.14 (Q5), R1.7 (D5), R2.14 (Q5), R2.7 (D5), R3.14 (Q5), R3.7 (D5), R4.14 (Q5), R4.7 (D5)
- net D6: now reaches J1.17 (Pin_17)
- net D6: now also B_IN1.12 (B6), B_OUT0.8 (A6), R0.13 (Q6), R0.8 (D6), R1.13 (Q6), R1.8 (D6), R2.13 (Q6), R2.8 (D6), R3.13 (Q6), R3.8 (D6), R4.13 (Q6), R4.8 (D6)
- net D7: now reaches J1.18 (Pin_18)
- net D7: now also B_IN1.11 (B7), B_OUT0.9 (A7), R0.12 (Q7), R0.9 (D7), R1.12 (Q7), R1.9 (D7), R2.12 (Q7), R2.9 (D7), R3.12 (Q7), R3.9 (D7), R4.12 (Q7), R4.9 (D7)
- net ZeroIn: now reaches J1.21 (Pin_21)
- net ZeroIn: now also B_IN0.11 (B7)
- net ~{CarryIn}: now reaches J1.22 (Pin_22)
- net ~{CarryIn}: now also B_IN0.12 (B6)
- net SignIn: now reaches J1.23 (Pin_23)
- net SignIn: now also B_IN0.13 (B5)
- removed net ALU0: B_IN0.11 (B7), J1.10 (Pin_10)
- net ALU1 renamed D0
- net D0: now also B_IN1.18 (B0), B_OUT0.2 (A0), R0.19 (Q0), R0.2 (D0), R1.19 (Q0), R1.2 (D0), R2.19 (Q0), R2.2 (D0), R3.19 (Q0), R3.2 (D0), R4.19 (Q0), R4.2 (D0); no longer B_IN0.12 (B6)
- net ALU2 renamed D1
- net D1: now also B_IN1.17 (B1), B_OUT0.3 (A1), R0.18 (Q1), R0.3 (D1), R1.18 (Q1), R1.3 (D1), R2.18 (Q1), R2.3 (D1), R3.18 (Q1), R3.3 (D1), R4.18 (Q1), R4.3 (D1); no longer B_IN0.13 (B5)
- net LOAD_FR renamed ~{LOAD_FR}
- net ~{LOAD_FR}: now also U4.3
- net LOAD_R0 renamed ~{LOAD_R0}
- net ~{LOAD_R0}: now also U1.2
- net LOAD_R1 renamed ~{LOAD_R1}
- net ~{LOAD_R1}: now also U3.2
- net LOAD_R2 renamed ~{LOAD_R2}
- net ~{LOAD_R2}: now also U1.8
- net LOAD_R3 renamed ~{LOAD_R3}
- net ~{LOAD_R3}: now also U1.11
- net LOAD_R4 renamed ~{LOAD_R4}
- net ~{LOAD_R4}: now also U1.5
- net OUT_R0 renamed ~{OUT_R0}
- net OUT_R1 renamed ~{OUT_R1}
- net OUT_R2 renamed ~{OUT_R2}
- net OUT_R3 renamed ~{OUT_R3}
- net OUT_R4 renamed ~{OUT_R4}
- new net: U3.6, U4.4
- new net: U3.5, U4.6
- new net: U3.4, U3.9
- no-connect marks 28 -> 25
Other:
- moved on the sheet: B_IN0, C1, C2, C3, C4, C5, C8, C9
