File: schematics/pointer_hub/pointer_hub.kicad_sch (KiCad schematic)
At the start: 34 parts, among them J3 Conn_02x25_Counter_Clockwise, U1 74HC193, U10 74HC245, U11 74HC193, U12 74HC193, U13 74HC193, U14 74HC193, U2 74HC193, U3 74HC193, U4 74HC245, U5 74HC193, U6 74HC245, U7 74HC00, U8 74HC245, U9 74HC00

Commit message: added lowarg to pointerhub, also replaced resistor + vcc logic by grnd and changing A and B pins(A was in became out...)
Parts:
- removed R1, R2, R3, R4: R, Resistor_THT:R_Axial_DIN0204_L3.6mm_D1.6mm_P7.62mm_Horizontal, symbol Device:R
- removed U1, U11, U12, U13, U14, U2, U3, U5: 74HC193, Package_DIP:DIP-16_W7.62mm_Socket_LongPads, symbol 74xx:74HC193
- removed U10, U4, U6, U8: 74HC245, Package_DIP:DIP-20_W7.62mm_Socket_LongPads, symbol 74xx:74HC245
- removed U7, U9: 74HC00, Package_SO:SOIC-14_3.9x8.7mm_P1.27mm, symbol 74xx:74HC00
- added C16, C17, C18: C, Capacitor_THT:CP_Radial_D4.0mm_P1.50mm, symbol Device:C
- added U1, U11, U12, U16, U17, U2, U3, U5: 74LS193, Package_DIP:DIP-16_W7.62mm_Socket_LongPads, symbol 74xx:74LS193
- added U10, U13, U14, U15, U4: 74LS245, Package_DIP:DIP-20_W7.62mm_Socket_LongPads, symbol 74xx:74LS245
- added U6, U8: 74LS00, Package_DIP:DIP-14_W7.62mm_Socket_LongPads, symbol 74xx:74LS00
- added U7: 74LS574, Package_DIP:DIP-20_W7.62mm_Socket_LongPads, symbol 74xx:74LS574
- added U9: 74LS08, Package_DIP:DIP-14_W7.62mm_Socket_LongPads, symbol 74xx:74LS08
- J3: footprint Connector_Harwin:Harwin_Gecko-G125-FVX5005L0X_2x25_P1.25mm_Vertical -> Connector_PinSocket_2.54mm:PinSocket_2x25_P2.54mm_Horizontal
Connections:
- net CLK is gone; now on net GND: J3.2 (Pin_2)
- net SPReset is gone; now on net BUS1: J3.12 (Pin_12)
- net ~CLK is gone; now on net GND: J3.49 (Pin_49)
- net ~SPHighOut is gone; now on net BUS7: J3.18 (Pin_18)
- net ~SPLowOut is gone; now on net BUS6: J3.17 (Pin_17)
- net BUS0: now also J3.11 (Pin_11), U10.2 (A0), U12.15 (A), U13.2 (A0), U14.2 (A0), U15.2 (A0), U2.15 (A), U3.15 (A), U4.2 (A0), U5.15 (A), U7.2 (D0); no longer J3.4 (Pin_4)
- net BUS1: now also U10.3 (A1), U12.1 (B), U13.3 (A1), U14.3 (A1), U15.3 (A1), U2.1 (B), U3.1 (B), U4.3 (A1), U5.1 (B), U7.3 (D1); no longer J3.5 (Pin_5)
- net BUS2: now also J3.13 (Pin_13), U10.4 (A2), U12.10 (C), U13.4 (A2), U14.4 (A2), U15.4 (A2), U2.10 (C), U3.10 (C), U4.4 (A2), U5.10 (C), U7.4 (D2); no longer J3.6 (Pin_6)
- net BUS3: now also J3.14 (Pin_14), U10.5 (A3), U12.9 (D), U13.5 (A3), U14.5 (A3), U15.5 (A3), U2.9 (D), U3.9 (D), U4.5 (A3), U5.9 (D), U7.5 (D3); no longer J3.7 (Pin_7)
- net BUS4: now also J3.15 (Pin_15), U1.15 (A), U10.6 (A4), U11.15 (A), U13.6 (A4), U14.6 (A4), U15.6 (A4), U16.15 (A), U17.15 (A), U4.6 (A4), U7.6 (D4); no longer J3.8 (Pin_8)
- net BUS5: now also J3.16 (Pin_16), U1.1 (B), U10.7 (A5), U11.1 (B), U13.7 (A5), U14.7 (A5), U15.7 (A5), U16.1 (B), U17.1 (B), U4.7 (A5), U7.7 (D5); no longer J3.9 (Pin_9)
- net BUS6: now also U1.10 (C), U10.8 (A6), U11.10 (C), U13.8 (A6), U14.8 (A6), U15.8 (A6), U16.10 (C), U17.10 (C), U4.8 (A6), U7.8 (D6); no longer J3.10 (Pin_10)
- net BUS7: now also U1.9 (D), U10.9 (A7), U11.9 (D), U13.9 (A7), U14.9 (A7), U15.9 (A7), U16.9 (D), U17.9 (D), U4.9 (A7), U7.9 (D7); no longer J3.11 (Pin_11)
- net CPd_A: now also U17.4 (DOWN), U6.6
- net CPd_B: now also U11.4 (DOWN), U8.8
- net CPu_A: now also U17.5 (UP), U6.3
- net CPu_B: now also U11.5 (UP), U8.11
- net DH_A0: now also U15.18 (B0), U2.3 (QA)
- net DH_A1: now also U15.17 (B1), U2.2 (QB)
- net DH_A2: now also U15.16 (B2), U2.6 (QC)
- net DH_A3: now also U15.15 (B3), U2.7 (QD)
- net DH_A4: now also U15.14 (B4), U16.3 (QA)
- net DH_A5: now also U15.13 (B5), U16.2 (QB)
- net DH_A6: now also U15.12 (B6), U16.6 (QC)
- net DH_A7: now also U15.11 (B7), U16.7 (QD)
- net DH_B0: now also U10.18 (B0), U5.3 (QA)
- net DH_B1: now also U10.17 (B1), U5.2 (QB)
- net DH_B2: now also U10.16 (B2), U5.6 (QC)
- net DH_B3: now also U10.15 (B3), U5.7 (QD)
- net DH_B4: now also U1.3 (QA), U10.14 (B4)
- net DH_B5: now also U1.2 (QB), U10.13 (B5)
- net DH_B6: now also U1.6 (QC), U10.12 (B6)
- net DH_B7: now also U1.7 (QD), U10.11 (B7)
- net DL_A0: now also U14.18 (B0), U3.3 (QA)
- net DL_A1: now also U14.17 (B1), U3.2 (QB)
- net DL_A2: now also U14.16 (B2), U3.6 (QC)
- net DL_A3: now also U14.15 (B3), U3.7 (QD)
- net DL_A4: now also U14.14 (B4), U17.3 (QA)
- net DL_A5: now also U14.13 (B5), U17.2 (QB)
- net DL_A6: now also U14.12 (B6), U17.6 (QC)
- net DL_A7: now also U14.11 (B7), U17.7 (QD)
- net DL_B0: now also U12.3 (QA), U4.18 (B0)
- net DL_B1: now also U12.2 (QB), U4.17 (B1)
- net DL_B2: now also U12.6 (QC), U4.16 (B2)
- net DL_B3: now also U12.7 (QD), U4.15 (B3)
- net DL_B4: now also U11.3 (QA), U4.14 (B4)
- net DL_B5: now also U11.2 (QB), U4.13 (B5)
- net DL_B6: now also U11.6 (QC), U4.12 (B6)
- net DL_B7: now also U11.7 (QD), U4.11 (B7)
- net GND: now also C1.1, C10.1, C11.1, C12.1, C13.1, C14.1, C2.1, C3.1, C4.1, C7.1, C9.1, J3.19 (Pin_19), C16.1, C17.1, C18.1, U1.8 (GND), U10.1 (A->B), U10.10 (GND), U11.8 (GND), U12.8 (GND), U13.1 (A->B), U13.10 (GND), U14.1 (A->B), U14.10 (GND), U15.10 (GND), U15.19 (CE), U16.8 (GND), U17.8 (GND), U2.8 (GND), U3.8 (GND), U4.1 (A->B), U4.10 (GND), U5.8 (GND), U6.7 (GND), U7.1 (OE), U7.10 (GND), U8.7 (GND), U9.7 (GND); no longer C1.2, C10.2, C11.2, C12.2, C13.2, C14.2, C2.2, C3.2, C4.2, C7.2, C9.2, J3.1 (Pin_1), J3.3 (Pin_3), J3.48 (Pin_48), J3.50 (Pin_50)
- net PCDec: now also U6.5
- net PCHighIn: now also U6.10
- net PCInc: now also U6.2
- net PCLowIn: now also U6.13
- net PULSE: now also J3.48 (Pin_48), U6.12, U6.9, U8.2, U8.5; no longer J3.47 (Pin_47)
- net Ph_A: now also U16.11 (~{LOAD}), U2.11 (~{LOAD}), U6.8
- net Ph_B: now also U1.11 (~{LOAD}), U5.11 (~{LOAD}), U8.6
- net Pl_A: now also U17.11 (~{LOAD}), U3.11 (~{LOAD}), U6.11
- net Pl_B: now also U11.11 (~{LOAD}), U12.11 (~{LOAD}), U8.3
- net SPDec: now also J3.41 (Pin_41), U8.9; no longer J3.14 (Pin_14)
- net SPHighIn: now also J3.42 (Pin_42), U8.4; no longer J3.15 (Pin_15)
- net SPInc: now also J3.40 (Pin_40), U8.12; no longer J3.13 (Pin_13)
- net SPLowIn: now also J3.43 (Pin_43), U8.1; no longer J3.16 (Pin_16)
- net VCC: now reaches J3.25 (Pin_25)
- net VCC: now also C1.2, C10.2, C11.2, C12.2, C13.2, C14.2, C15.2, C2.2, C3.2, C4.2, C5.1, C6.1, C7.2, C8.1, C9.2, J3.1 (Pin_1), J3.26 (Pin_26), J3.50 (Pin_50), C16.2, C17.2, C18.2, U1.16 (VCC), U10.20 (VCC), U11.16 (VCC), U12.16 (VCC), U13.20 (VCC), U14.20 (VCC), U15.20 (VCC), U16.16 (VCC), U17.16 (VCC), U2.16 (VCC), U3.16 (VCC), U4.20 (VCC), U5.16 (VCC), U6.14 (VCC), U7.20 (VCC), U8.14 (VCC), U9.14 (VCC)
- net ~{SPLowOut}: now reaches J3.44 (Pin_44)
- net ~{SPLowOut}: now also U4.19 (CE)
- net ~{SPHighOut}: now reaches J3.45 (Pin_45)
- net ~{SPHighOut}: now also U10.19 (CE)
- removed net +5V: C1.1, C10.1, C11.1, C12.1, C13.1, C14.1, C15.2, C2.1, C3.1, C4.1, C5.1, C6.1, C7.1, C8.1, C9.1
- net PCReset renamed Reset
- net Reset: now also U1.14 (CLR), U11.14 (CLR), U12.14 (CLR), U16.14 (CLR), U17.14 (CLR), U2.14 (CLR), U3.14 (CLR), U5.14 (CLR)
- net ~PСHighOut renamed ~{PСHighOut}
- net ~{PСHighOut}: now also U15.1 (A->B)
- net ~PСLowOut renamed ~{PСLowOut}
- net ~{PСLowOut}: now also U14.19 (CE)
- new net: U17.12 (~{CO}), U3.5 (UP)
- new net: U17.13 (~{BO}), U3.4 (DOWN)
- new net: U16.13 (~{BO}), U2.4 (DOWN)
- new net: U16.12 (~{CO}), U2.5 (UP)
- new net: U1.5 (UP), U12.12 (~{CO})
- new net: U1.4 (DOWN), U12.13 (~{BO})
- new net: U11.13 (~{BO}), U12.4 (DOWN)
- new net: U11.12 (~{CO}), U12.5 (UP)
- new net: U1.13 (~{BO}), U5.4 (DOWN)
- new net: U1.12 (~{CO}), U5.5 (UP)
- new net: U16.4 (DOWN), U3.13 (~{BO})
- new net: U16.5 (UP), U3.12 (~{CO})
- new net: U7.11 (Cp), U9.3
- new net: U13.11 (B7), U7.12 (Q7)
- new net: U13.12 (B6), U7.13 (Q6)
- new net: U13.13 (B5), U7.14 (Q5)
- new net: U13.14 (B4), U7.15 (Q4)
- new net: U13.15 (B3), U7.16 (Q3)
- new net: U13.16 (B2), U7.17 (Q2)
- new net: U13.17 (B1), U7.18 (Q1)
- new net: U13.18 (B0), U7.19 (Q0)
- new net Clk: J3.4 (Pin_4), U9.2
- new net LFromD: J3.5 (Pin_5), U9.1
- new net ~{Clk}: J3.3 (Pin_3), U6.1, U6.4, U8.10, U8.13
- new net ~{LToD}: J3.6 (Pin_6), U13.19 (CE)
- no-connect marks 25 -> 29
Other:
- moved on the sheet: C10, C12, C14, C2, C3, C8, J3
