File: schematics/alu/alu.kicad_sch (KiCad schematic)
At the start: 33 parts, among them J1 Conn_02x25_Counter_Clockwise, U1 74LS574, U10 74LS02, U11 74LS245, U12 74LS574, U13 74LS245, U2 74LS08, U3 74LS245, U4 74LS245, U5 74LS245, U6 74LS137, U7 74LS181, U8 74LS181, U9 74LS02

Commit message: fix(kicad): updated footprints
Other:
- company: HardServe Inc. -> (none)
Changed lines of the file:
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@@
 		(date "20/10/2025")
 		(rev "1.0.0")
-		(company "HardServe Inc.")
 	)
 	(junction
@@
 	)
 	(label "H5"
-		(at 199.39 36.83 180)
+		(at 198.12 36.83 180)
 		(effects
 			(font
@@
 	)
 	(label "H4"
-		(at 199.39 34.29 180)
+		(at 198.12 34.29 180)
 		(effects
 			(font
@@
 	)
 	(label "H7"
-		(at 199.39 41.91 180)
+		(at 198.12 41.91 180)
 		(effects
 			(font
@@
 	)
 	(label "H6"
-		(at 199.39 39.37 180)
+		(at 198.12 39.37 180)
 		(effects
 			(font
@@
 		)
 		(property "Type" "ShiftRight"
-			(at 370.84 128.27 0)
+			(at 370.84 123.952 0)
 			(effects
 				(font

Commit message: fix(kicad): added footprints
Parts:
- J1: footprint (none) -> Connector_PinSocket_2.54mm:PinSocket_2x25_P2.54mm_Horizontal
- U1, U11, U12, U13, U3, U4, U5: footprint (none) -> Package_DIP:DIP-20_W7.62mm_Socket_LongPads
- U10, U2, U9: footprint (none) -> Package_DIP:DIP-14_W7.62mm_Socket_LongPads
- U6: footprint (none) -> Package_DIP:DIP-16_W7.62mm_Socket_LongPads
- U7, U8: footprint (none) -> Package_DIP:DIP-24_18.0mmx34.29mm_W15.24mm_Socket_LongPads
Changed lines of the file:
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@@
 			)
 		)
-		(property "Footprint" ""
+		(property "Footprint" "Package_DIP:DIP-14_W7.62mm_Socket_LongPads"
 			(at 261.62 125.73 0)
 			(effects
@@
 			)
 		)
-		(property "Footprint" ""
+		(property "Footprint" "Package_DIP:DIP-14_W7.62mm_Socket_LongPads"
 			(at 245.11 134.62 0)
 			(effects
@@
 			)
 		)
-		(property "Footprint" ""
+		(property "Footprint" "Package_DIP:DIP-20_W7.62mm_Socket_LongPads"
 			(at 370.84 181.61 0)
 			(effects
@@
 			)
 		)
-		(property "Footprint" ""
+		(property "Footprint" "Package_DIP:DIP-14_W7.62mm_Socket_LongPads"
 			(at 74.93 49.53 0)
 			(effects
@@
 			)
 		)
-		(property "Footprint" ""
+		(property "Footprint" "Package_DIP:DIP-14_W7.62mm_Socket_LongPads"
 			(at 96.52 201.93 0)
 			(effects
@@
 			)
 		)
-		(property "Footprint" ""
+		(property "Footprint" "Package_DIP:DIP-14_W7.62mm_Socket_LongPads"
 			(at 281.94 100.33 0)
 			(effects
@@
 			)
 		)
-		(property "Footprint" ""
+		(property "Footprint" "Package_DIP:DIP-14_W7.62mm_Socket_LongPads"
 			(at 148.59 264.16 0)
 			(effects
@@
 			)
 		)
-		(property "Footprint" ""
+		(property "Footprint" "Package_DIP:DIP-24_18.0mmx34.29mm_W15.24mm_Socket_LongPads"
 			(at 213.36 52.07 0)
 			(effects
@@
 			)
 		)
-		(property "Footprint" ""
+		(property "Footprint" "Package_DIP:DIP-14_W7.62mm_Socket_LongPads"
 			(at 22.86 264.16 0)
 			(effects
@@
 			)
 		)
-		(property "Footprint" ""
+		(property "Footprint" "Package_DIP:DIP-16_W7.62mm_Socket_LongPads"
 			(at 328.93 176.53 0)
 			(effects
@@
 			)
 		)
-		(property "Footprint" ""
+		(property "Footprint" "Connector_PinSocket_2.54mm:PinSocket_2x25_P2.54mm_Horizontal"
 			(at 35.56 69.85 0)
 			(effects
@@
 			)
 		)
-		(property "Footprint" ""
+		(property "Footprint" "Package_DIP:DIP-14_W7.62mm_Socket_LongPads"
 			(at 261.62 77.47 0)
 			(effects
@@
 			)
 		)
-		(property "Footprint" ""
+		(property "Footprint" "Package_DIP:DIP-20_W7.62mm_Socket_LongPads"
 			(at 370.84 228.6 0)
 			(effects
@@
 			)
 		)
-		(property "Footprint" ""
+		(property "Footprint" "Package_DIP:DIP-14_W7.62mm_Socket_LongPads"
 			(at 245.11 86.36 0)
 			(effects
@@
 			)
 		)
-		(property "Footprint" ""
+		(property "Footprint" "Package_DIP:DIP-14_W7.62mm_Socket_LongPads"
 			(at 245.11 118.11 0)
 			(effects
@@
 			)
 		)
-		(property "Footprint" ""
+		(property "Footprint" "Package_DIP:DIP-14_W7.62mm_Socket_LongPads"
 			(at 297.18 100.33 0)
 			(effects
@@
 			)
 		)
-		(property "Footprint" ""
+		(property "Footprint" "Package_DIP:DIP-14_W7.62mm_Socket_LongPads"
 			(at 245.11 68.58 0)
 			(effects
@@
 			)
 		)
-		(property "Footprint" ""
+		(property "Footprint" "Package_DIP:DIP-20_W7.62mm_Socket_LongPads"
 			(at 100.33 35.56 0)
 			(effects
@@
 			)
 		)
-		(property "Footprint" ""
+		(property "Footprint" "Package_DIP:DIP-14_W7.62mm_Socket_LongPads"
 			(at 91.44 264.16 0)
 			(effects
@@
 			)
 		)
-		(property "Footprint" ""
+		(property "Footprint" "Package_DIP:DIP-14_W7.62mm_Socket_LongPads"
 			(at 57.15 264.16 0)
 			(effects
@@
 			)
 		)
-		(property "Footprint" ""
+		(property "Footprint" "Package_DIP:DIP-20_W7.62mm_Socket_LongPads"
 			(at 151.13 210.82 0)
 			(effects
@@
 			)
 		)
-		(property "Footprint" ""
+		(property "Footprint" "Package_DIP:DIP-24_18.0mmx34.29mm_W15.24mm_Socket_LongPads"
 			(at 163.83 80.01 0)
 			(effects
@@
 			)
 		)
-		(property "Footprint" ""
+		(property "Footprint" "Package_DIP:DIP-20_W7.62mm_Socket_LongPads"
 			(at 341.63 86.36 0)
 			(effects
@@
 			)
 		)
-		(property "Footprint" ""
+		(property "Footprint" "Package_DIP:DIP-20_W7.62mm_Socket_LongPads"
 			(at 370.84 128.27 0)
 			(effects
@@
 			)
 		)
-		(property "Footprint" ""
+		(property "Footprint" "Package_DIP:DIP-20_W7.62mm_Socket_LongPads"
 			(at 198.12 204.47 0)
 			(effects
@@
 			)
 		)
-		(property "Footprint" ""
+		(property "Footprint" "Package_DIP:DIP-14_W7.62mm_Socket_LongPads"
 			(at 163.83 264.16 0)
 			(effects

Commit message: fix(kicad): fixed kicad ERC errors, replaces resistors to capacitors
Parts:
- removed R10, R11, R12, R13, R14, R15, R16, R5, R6, R7, R8, R9: R, symbol Device:R
- removed U1: 74LS574, Package_DIP:DIP-20_W7.62mm_Socket_LongPads, symbol 74xx:74LS574
- added C10, C11, C12, C13, C4, C5, C6, C7, C8, C9: C, symbol Device:C
- added U14: 74LS574, symbol 74xx:74LS574
Connections:
- net ACCUM0: now also U14.19 (Q0)
- net ACCUM1: now also U14.18 (Q1)
- net ACCUM2: now also U14.17 (Q2)
- net ACCUM3: now also U14.16 (Q3)
- net ACCUM4: now also U14.15 (Q4)
- net ACCUM5: now also U14.14 (Q5)
- net ACCUM6: now also U14.13 (Q6)
- net ACCUM7: now also U14.12 (Q7)
- net BUS0: now also U11.2 (A0), U13.2 (A0), U14.2 (D0); no longer U11.18 (B0), U13.18 (B0)
- net BUS1: now also U11.3 (A1), U13.3 (A1), U14.3 (D1); no longer U11.17 (B1), U13.17 (B1)
- net BUS2: now also U11.4 (A2), U13.4 (A2), U14.4 (D2); no longer U11.16 (B2), U13.16 (B2)
- net BUS3: now also U11.5 (A3), U13.5 (A3), U14.5 (D3); no longer U11.15 (B3), U13.15 (B3)
- net BUS4: now also U11.6 (A4), U13.6 (A4), U14.6 (D4); no longer U11.14 (B4), U13.14 (B4)
- net BUS5: now also U11.7 (A5), U13.7 (A5), U14.7 (D5); no longer U11.13 (B5), U13.13 (B5)
- net BUS6: now also U11.8 (A6), U13.8 (A6), U14.8 (D6); no longer U11.12 (B6), U13.12 (B6)
- net BUS7: now also U11.9 (A7), U13.9 (A7), U14.9 (D7); no longer U11.11 (B7), U13.11 (B7)
- net GND: now also U11.1 (A->B), U12.1 (OE), U12.10 (GND), U13.1 (A->B), C10.1, C11.1, C12.2, C13.2, C4.1, C5.1, C6.2, C7.1, C8.2, C9.2, U14.1 (OE), U14.10 (GND)
- net H0: now also U13.18 (B0); no longer U13.2 (A0)
- net H1: now also U13.17 (B1); no longer U13.3 (A1)
- net H2: now also U13.16 (B2); no longer U13.4 (A2)
- net H3: now also U13.15 (B3); no longer U13.5 (A3)
- net H4: now also U13.14 (B4); no longer U13.6 (A4)
- net H5: now also U13.13 (B5); no longer U13.7 (A5)
- net H6: now also U13.12 (B6); no longer U13.8 (A6)
- net H7: now also U13.11 (B7); no longer U13.9 (A7)
- net Sign: now also U11.11 (B7); no longer U11.9 (A7)
- net VCC: now also U11.20 (VCC), U12.20 (VCC), U13.20 (VCC), U3.20 (VCC), U4.20 (VCC), U5.20 (VCC), U6.16 (VCC), U7.24 (VCC), U8.24 (VCC), C10.2, C11.2, C12.1, C13.1, C4.2, C5.2, C6.1, C7.2, C8.1, C9.1, U14.20 (VCC)
- net at U7.11 (F2), U9.5: now also U11.16 (B2); no longer U11.4 (A2)
- net at U7.13 (F3), U9.6: now also U11.15 (B3); no longer U11.5 (A3)
- net at U2.3: now also U14.11 (Cp)
- net at U10.9, U8.10 (F1): now also U11.13 (B5); no longer U11.7 (A5)
- net at U8.11 (F2), U9.11: now also U11.12 (B6); no longer U11.8 (A6)
- net at U10.8, U8.9 (F0): now also U11.14 (B4); no longer U11.6 (A4)
- net at U7.9 (F0), U9.2: now also U11.18 (B0); no longer U11.2 (A0)
- net at U7.10 (F1), U9.3: now also U11.17 (B1); no longer U11.3 (A1)

Commit message: Connnect all modules together
Parts:
- removed U2: 74LS08, Package_DIP:DIP-14_W7.62mm_Socket_LongPads, symbol 74xx:74LS08
- added U1: 74LS02, symbol 74xx:74LS02
- U14: footprint (none) -> Package_DIP:DIP-20_W7.62mm_Socket_LongPads
- U7, U8: footprint Package_DIP:DIP-24_18.0mmx34.29mm_W15.24mm_Socket_LongPads -> Package_DIP:DIP-24_W7.62mm_Socket_LongPads
Connections:
- net GND: now also U1.7 (GND)
- net VCC: now also U1.14 (VCC)
- net ~{Clk}: now also U1.3, U1.6
- net at U14.11 (Cp): now also U1.1
- net at U12.11 (Cp): now also U1.4
- net Clk: no longer names the net of J1.4 (Pin_4)
- net FromD renamed ~{FromD}
- net ~{FromD}: now also U1.2
- net HFromD renamed ~{HFromD}
- net ~{HFromD}: now also U1.5
- net ToD renamed ~{ToD}
