File: schematics/gen2/interface/interface.kicad_sch (KiCad schematic)
At the start: 16 parts, among them U1 74LS00, U2 74LS00, U4 74LS245, U5 74LS193, U6 74LS193, U7 74LS193, U8 74LS193

Commit message: Implement code changes to enhance functionality and improve performance
Parts:
- added C8: C, Capacitor_THT:C_Radial_D6.3mm_H5.0mm_P2.50mm, symbol Device:C
- C1, C2, C3, C4, C5, C6, C7: footprint Capacitor_SMD:C_0805_2012Metric_Pad1.18x1.45mm_HandSolder -> Capacitor_THT:C_Disc_D5.0mm_W2.5mm_P5.00mm
Connections:
- net GND: now also C1.2, C2.2, C3.2, C4.2, C5.2, C6.2, C7.2, C8.2; no longer C1.1, C2.1, C3.1, C4.1, C5.1, C6.1, C7.1
- net VCC: now also C1.1, C2.1, C3.1, C4.1, C5.1, C6.1, C7.1, C8.1; no longer C1.2, C2.2, C3.2, C4.2, C5.2, C6.2, C7.2

Commit message: fix(kicad): vcc zones
Parts:
- PAD2: footprint Connector_PinSocket_2.54mm:PinSocket_2x19_P2.54mm_Horizontal -> Connector_PinSocket_2.54mm:PinSocket_2x19_P2.54mm_Vertical
Changed lines of the file:
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@@
 			)
 		)
-		(property "Footprint" "Connector_PinSocket_2.54mm:PinSocket_2x19_P2.54mm_Horizontal"
+		(property "Footprint" "Connector_PinSocket_2.54mm:PinSocket_2x19_P2.54mm_Vertical"
 			(at 220.98 41.91 0)
 			(effects
