File: schematics/core_1/core_1.kicad_pcb (KiCad board)
At the start: 2 copper layers, 100 x 91.1 mm, 22 parts, among them U1 74LS00, U2 74LS04, U3 74LS109, U4 74LS02

Commit message: silklayer check
Parts:
- moved kibuzzard-6911CC41 9.12 mm to (108.2, 57.3)
Routing:
- net Net-(DECODER3-E1): track 164.7 -> 158.7 mm
