File: schematics/register_file_accum/register_file_accum.kicad_sch (KiCad schematic)
At the start: 31 parts, among them U1 74LS02, U2 74LS02, U3 74LS02, U4 74LS138, U5 74LS574, U6 74LS245, U7 74LS245, U8 74LS245

Commit message: Add test points
Parts:
- added TP1: ~{ReadZH}, Connector_Pin:Pin_D1.0mm_L10.0mm, symbol Connector:TestPoint
- added TP10: ~{ReadXH}, Connector_Pin:Pin_D1.0mm_L10.0mm, symbol Connector:TestPoint
- added TP11: ~{LoadXL}, Connector_Pin:Pin_D1.0mm_L10.0mm, symbol Connector:TestPoint
- added TP12: ~{PassXL}, Connector_Pin:Pin_D1.0mm_L10.0mm, symbol Connector:TestPoint
- added TP13: ~{LeftXL}, Connector_Pin:Pin_D1.0mm_L10.0mm, symbol Connector:TestPoint
- added TP14: ~{RightXL}, Connector_Pin:Pin_D1.0mm_L10.0mm, symbol Connector:TestPoint
- added TP15: ~{Clock}, Connector_Pin:Pin_D1.0mm_L10.0mm, symbol Connector:TestPoint
- added TP16: Power, Connector_Pin:Pin_D1.0mm_L10.0mm, symbol Connector:TestPoint
- added TP2: ~{LoadZH}, Connector_Pin:Pin_D1.0mm_L10.0mm, symbol Connector:TestPoint
- added TP3: ~{LoadZL}, Connector_Pin:Pin_D1.0mm_L10.0mm, symbol Connector:TestPoint
- added TP4: ~{ReadZL}, Connector_Pin:Pin_D1.0mm_L10.0mm, symbol Connector:TestPoint
- added TP5: ~{LoadYH}, Connector_Pin:Pin_D1.0mm_L10.0mm, symbol Connector:TestPoint
- added TP6: ~{ReadYH}, Connector_Pin:Pin_D1.0mm_L10.0mm, symbol Connector:TestPoint
- added TP7: ~{LoadYL}, Connector_Pin:Pin_D1.0mm_L10.0mm, symbol Connector:TestPoint
- added TP8: ~{ReadYL}, Connector_Pin:Pin_D1.0mm_L10.0mm, symbol Connector:TestPoint
- added TP9: ~{LoadXH}, Connector_Pin:Pin_D1.0mm_L10.0mm, symbol Connector:TestPoint
Connections:
- net ACSHLEFT: now also TP13.1
- net ACSHRIGHT: now also TP14.1
- net VCC: now also TP16.1
- net ~{CLK}: now also TP15.1
- net ~{RAC}: now also TP12.1
- net at R2.11 (Cp), U1.10: now also TP5.1
- net at R4.11 (Cp), U1.4: now also TP9.1
- net at BC1.B27 (~{RZH}), R0.1 (OE): now also TP1.1
- net at R0.11 (Cp), U1.1: now also TP2.1
- net at BC1.B22 (~{RXH}), R4.1 (OE): now also TP10.1
- net at BC1.B24 (~{RYL}), R3.1 (OE): now also TP8.1
- net at BC1.B26 (~{RZL}), R1.1 (OE): now also TP4.1
- net at R3.11 (Cp), U1.13: now also TP7.1
- net at R1.11 (Cp), U2.1: now also TP3.1
- net at U3.1, U5.11 (Cp): now also TP11.1

Commit message: Add test points for register file + accum
Parts:
- Power1: renamed from TP16; footprint Connector_Pin:Pin_D1.0mm_L10.0mm -> TestPoint:TestPoint_Pad_D1.0mm
- ~{Clock}1: renamed from TP15; footprint Connector_Pin:Pin_D1.0mm_L10.0mm -> TestPoint:TestPoint_Pad_D1.0mm
- ~{LeftXL}1: renamed from TP13; footprint Connector_Pin:Pin_D1.0mm_L10.0mm -> TestPoint:TestPoint_Pad_D1.0mm
- ~{LoadXH}1: renamed from TP9; footprint Connector_Pin:Pin_D1.0mm_L10.0mm -> TestPoint:TestPoint_Pad_D1.0mm
- ~{LoadXL}1: renamed from TP11; footprint Connector_Pin:Pin_D1.0mm_L10.0mm -> TestPoint:TestPoint_Pad_D1.0mm
- ~{LoadYH}1: renamed from TP5; footprint Connector_Pin:Pin_D1.0mm_L10.0mm -> TestPoint:TestPoint_Pad_D1.0mm
- ~{LoadYL}1: renamed from TP7; footprint Connector_Pin:Pin_D1.0mm_L10.0mm -> TestPoint:TestPoint_Pad_D1.0mm
- ~{LoadZH}1: renamed from TP2; footprint Connector_Pin:Pin_D1.0mm_L10.0mm -> TestPoint:TestPoint_Pad_D1.0mm
- ~{LoadZL}1: renamed from TP3; footprint Connector_Pin:Pin_D1.0mm_L10.0mm -> TestPoint:TestPoint_Pad_D1.0mm
- ~{PassXL}1: renamed from TP12; footprint Connector_Pin:Pin_D1.0mm_L10.0mm -> TestPoint:TestPoint_Pad_D1.0mm
- ~{ReadXH}1: renamed from TP10; footprint Connector_Pin:Pin_D1.0mm_L10.0mm -> TestPoint:TestPoint_Pad_D1.0mm
- ~{ReadYH}1: renamed from TP6; footprint Connector_Pin:Pin_D1.0mm_L10.0mm -> TestPoint:TestPoint_Pad_D1.0mm
- ~{ReadYL}1: renamed from TP8; footprint Connector_Pin:Pin_D1.0mm_L10.0mm -> TestPoint:TestPoint_Pad_D1.0mm
- ~{ReadZH}1: renamed from TP1; footprint Connector_Pin:Pin_D1.0mm_L10.0mm -> TestPoint:TestPoint_Pad_D1.0mm
- ~{ReadZL}1: renamed from TP4; footprint Connector_Pin:Pin_D1.0mm_L10.0mm -> TestPoint:TestPoint_Pad_D1.0mm
- ~{RightXL}1: renamed from TP14; footprint Connector_Pin:Pin_D1.0mm_L10.0mm -> TestPoint:TestPoint_Pad_D1.0mm
- renumbered R4 to XH1, U5 to XL1, R2 to YH1, R3 to YL1, R0 to ZH1, R1 to ZL1
Connections:
- net at BC1.B25 (~{RYH}), YH1.1 (OE): now also ~{ReadYH}1.1
Other:
- moved on the sheet: Power1, ~{ReadYH}1
