File: schematics/core_2/core_2.kicad_pcb (KiCad board)
At the start: 2 copper layers, 100 x 91.1 mm, 36 parts, among them U1 74LS04, U2 74LS574, U3 74LS02, U5 74LS00

Commit message: fix
Parts:
- removed CARRY, CP, SIGN, VCC, ZERO, carry, clk, sign, zero: TestPoint, TestPoint:TestPoint_Pad_D1.0mm
- removed load FR: TestPoint, TestPoint:TestPoint_Pad_D1.0mm
- removed out FR: TestPoint, TestPoint:TestPoint_Pad_D1.0mm
- removed update FR: TestPoint, TestPoint:TestPoint_Pad_D1.0mm
- added CarryO1: TestPoint, TestPoint:TestPoint_Pad_D1.0mm, F.Cu at (251.1, 38.9)
- added PWR1: TestPoint, TestPoint:TestPoint_Pad_D1.0mm, F.Cu at (190.5, 99.5)
- added SignO1: TestPoint, TestPoint:TestPoint_Pad_D1.0mm, F.Cu at (248.1, 38.4)
- added ZerroIn1: TestPoint, TestPoint:TestPoint_Pad_D1.0mm, F.Cu at (265.2, 94.4)
- added ZerroO1: TestPoint, TestPoint:TestPoint_Pad_D1.0mm, F.Cu at (253.7, 38.9)
- added kibuzzard-691DDE8A: G***, kibuzzard-691DDE8A, F.Cu at (222.9, 14.1)
- added ~{CLK}1: TestPoint, TestPoint:TestPoint_Pad_D1.0mm, F.Cu at (281.0, 98.5)
- added ~{CarrIn}1: TestPoint, TestPoint:TestPoint_Pad_D1.0mm, F.Cu at (263.4, 93.2)
- added ~{ENBL}1: TestPoint, TestPoint:TestPoint_Pad_D1.0mm, F.Cu at (275.6, 40.6)
- added ~{L_FR}1: TestPoint, TestPoint:TestPoint_Pad_D1.0mm, F.Cu at (199.5, 74.0)
- added ~{OUT_FR}1: TestPoint, TestPoint:TestPoint_Pad_D1.0mm, F.Cu at (190.2, 73.7)
- added ~{SignIn}1: TestPoint, TestPoint:TestPoint_Pad_D1.0mm, F.Cu at (261.7, 91.9)
- added ~{UPD_FR}1: TestPoint, TestPoint:TestPoint_Pad_D1.0mm, F.Cu at (238.5, 84.0)
Routing:
- net /~{OUT_FR}: track 144.9 -> 116.8 mm
- net /STATE8: track 136.7 -> 125.5 mm
- net /~{LOAD_FR}: track 163.8 -> 153.9 mm, vias 17 -> 16
- net /STATE9: track 139.7 -> 132.0 mm
- net /~{UPDATE_FR}: track 121.5 -> 114.7 mm, vias 9 -> 8
- net Net-(U2-Cp): track 35.4 -> 29.9 mm
- net /STATE10: track 153.1 -> 148.1 mm
- net /ZeroIn: track 38.8 -> 34.0 mm
- net /~{CarryIn}: track 41.8 -> 37.6 mm
- net /~CLK: track 148.2 -> 144.5 mm
- net /SignIn: track 34.8 -> 32.4 mm
