File: schematics/core_2/core_2.kicad_pcb (KiCad board)
At the start: 2 copper layers, 100 x 91.1 mm, 37 parts, among them U1 74LS04, U2 74LS574, U3 74LS02, U5 74LS00

Commit message: done
Parts:
- added kibuzzard-691DE0EC: G***, kibuzzard-691DE0EC, F.Cu at (272.0, 68.0)
