File: schematics/stack_pointer/step_counter.kicad_pcb (KiCad board)
At the start: 2 copper layers, 100 x 91 mm, 28 parts, among them U1 74HC00, U2 74HC193, U3 74HC193, U4 74HC193, U5 74HC193, U6 74HC245, U7 74HC245

Commit message: done
Parts:
- added kibuzzard-691DE1DA: G***, kibuzzard-691DE1DA, F.Cu at (199.0, 84.5)
Changed lines of the file:
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@@
 				(font
 					(size 0.001 0.001)
+					(thickness 0.15)
 				)
 			)
@@
 				(font
 					(size 0.001 0.001)
+					(thickness 0.15)
 				)
 			)
@@
 		)
 	)
+	(footprint "kibuzzard-691DE1DA"
+		(layer "F.Cu")
+		(at 199 84.5 90)
+		(descr "Generated with KiBuzzard")
+		(tags "kb_params=eyJBbGlnbm1lbnRDaG9pY2UiOiAiQ2VudGVyIiwgIkNhcExlZnRDaG9pY2UiOiAiIiwgIkNhcFJpZ2h0Q2hvaWNlIjogIi8iLCAiRm9udENvbWJvQm94IjogIlRvdXJuZXktUmVndWxhciIsICJIZWlnaHRDdHJsIjogMi4wLCAiTGF5ZXJDb21ib0JveCI6ICJGLlNpbGtTIiwgIkxpbmVTcGFjaW5nQ3RybCI6IDEuNSwgIk11bHRpTGluZVRleHQiOiAiYmViZWJlIiwgIlBhZGRpbmdCb3R0b21DdHJsIjogNS4wLCAiUGFkZGluZ0xlZnRDdHJsIjogNS4wLCAiUGFkZGluZ1JpZ2h0Q3RybCI6IDUuMCwgIlBhZGRpbmdUb3BDdHJsIjogNS4wLCAiV2lkdGhDdHJsIjogMi4wLCAiYWR2YW5jZWRDaGVja2JveCI6IHRydWUsICJpbmxpbmVGb3JtYXRUZXh0Ym94IjogdHJ1ZSwgImxpbmVvdmVyU3R5bGVDaG9pY2UiOiAiU3F1YXJlIiwgImxpbmVvdmVyVGhpY2tuZXNzQ3RybCI6IDF9")
+		(property "Reference" "kibuzzard-691DE1DA"
+			(at 0 -4.119429 90)
+			(layer "F.SilkS")
+			(hide yes)
+			(effects
+				(font
+					(size 0.001 0.001)
+					(thickness 0.15)
+				)
+			)
+		)
+		(property "Value" "G***"
+			(at 0 4.119429 90)
+			(layer "F.SilkS")
+			(hide yes)
+			(effects
+				(font
+					(size 0.001 0.001)
+					(thickness 0.15)
+				)
+			)
+		)
+		(property "Datasheet" ""
+			(at 0 0 90)
+			(layer "F.Fab")
+			(hide yes)
+			(effects
+				(font
+					(size 1.27 1.27)
+					(thickness 0.15)
+				)
+			)
+		)
+		(property "Description" ""
+			(at 0 0 90)
+			(layer "F.Fab")
+			(hide yes)
+			(effects
+				(font
+					(size 1.27 1.27)
+					(thickness 0.15)
+				)
+			)
+		)
+		(attr board_only exclude_from_pos_files exclude_from_bom)
+		(fp_poly
+			(pts
+				(xy 4.670714 -0.178571) (xy 4.817857 -0.032857) (xy 4.817857 0.118571) (xy 4.693571 0.242857) (xy 4.040714 0.242857)
+				(xy 4.040714 0.134286) (xy 4.649286 0.134286) (xy 4.709286 0.074286) (xy 4.709286 0.02) (xy 4.620714 -0.067143)
+				(xy 4.127857 -0.067143) (xy 4.040714 0.02) (xy 4.040714 0.134286) (xy 4.040714 0.242857) (xy 3.922143 0.242857)
+				(xy 3.922143 -0.025714) (xy 4.075 -0.178571) (xy 4.670714 -0.178571)
+			)
+			(stroke
+				(width 0)
+				(type solid)
+			)
+			(fill yes)
+			(layer "F.SilkS")
+		)
+		(fp_poly
+			(pts
+				(xy 1.150714 -0.178571) (xy 1.297857 -0.032857) (xy 1.297857 0.118571) (xy 1.173571 0.242857) (xy 0.520714 0.242857)
+				(xy 0.520714 0.134286) (xy 1.129286 0.134286) (xy 1.189286 0.074286) (xy 1.189286 0.02) (xy 1.100714 -0.067143)
+				(xy 0.607857 -0.067143) (xy 0.520714 0.02) (xy 0.520714 0.134286) (xy 0.520714 0.242857) (xy 0.402143 0.242857)
+				(xy 0.402143 -0.025714) (xy 0.555 -0.178571) (xy 1.150714 -0.178571)
+			)
+			(stroke
+				(width 0)
+				(type solid)
+			)
+			(fill yes)
+			(layer "F.SilkS")
+		)
+		(fp_poly
+			(pts
+				(xy -2.369286 -0.178571) (xy -2.222143 -0.032857) (xy -2.222143 0.118571) (xy -2.346429 0.242857)
+				(xy -2.999286 0.242857) (xy -2.999286 0.134286) (xy -2.390714 0.134286) (xy -2.330714 0.074286)
+				(xy -2.330714 0.02) (xy -2.419286 -0.067143) (xy -2.912143 -0.067143) (xy -2.999286 0.02) (xy -2.999286 0.134286)
+				(xy -2.999286 0.242857) (xy -3.117857 0.242857) (xy -3.117857 -0.025714) (xy -2.965 -0.178571) (xy -2.369286 -0.178571)
+			)
+			(stroke
+				(width 0)
+				(type solid)
+			)
+			(fill yes)
+			(layer "F.SilkS")
+		)
+		(fp_poly
+			(pts
+				(xy 2.375 0.781429) (xy 2.220714 0.628571) (xy 2.220714 0.008571) (xy 2.413571 -0.182857) (xy 2.886429 -0.182857)
+				(xy 3.026429 -0.045714) (xy 3.026429 0.628571) (xy 2.872143 0.781429) (xy 2.419286 0.781429) (xy 2.419286 0.667143)
+				(xy 2.830714 0.667143) (xy 2.917857 0.58) (xy 2.917857 0.02) (xy 2.830714 -0.068571) (xy 2.446429 -0.068571)
+				(xy 2.332143 0.047143) (xy 2.332143 0.58) (xy 2.419286 0.667143) (xy 2.419286 0.781429) (xy 2.375 0.781429)
+			)
+			(stroke
+				(width 0)
+				(type solid)
+			)
+			(fill yes)
+			(layer "F.SilkS")
+		)
+		(fp_poly
+			(pts
+				(xy -1.145 0.781429) (xy -1.299286 0.628571) (xy -1.299286 0.008571) (xy -1.106429 -0.182857) (xy -0.633571 -0.182857)
+				(xy -0.493571 -0.045714) (xy -0.493571 0.628571) (xy -0.647857 0.781429) (xy -1.100714 0.781429)
+				(xy -1.100714 0.667143) (xy -0.689286 0.667143) (xy -0.602143 0.58) (xy -0.602143 0.02) (xy -0.689286 -0.068571)
+				(xy -1.073571 -0.068571) (xy -1.187857 0.047143) (xy -1.187857 0.58) (xy -1.100714 0.667143) (xy -1.100714 0.781429)
+				(xy -1.145 0.781429)
+			)
+			(stroke
+				(width 0)
+				(type solid)
+			)
+			(fill yes)
+			(layer "F.SilkS")
+		)
+		(fp_poly
+			(pts
+				(xy -4.665 0.781429) (xy -4.819286 0.628571) (xy -4.819286 0.008571) (xy -4.626429 -0.182857) (xy -4.153571 -0.182857)
+				(xy -4.013571 -0.045714) (xy -4.013571 0.628571) (xy -4.167857 0.781429) (xy -4.620714 0.781429)
+				(xy -4.620714 0.667143) (xy -4.209286 0.667143) (xy -4.122143 0.58) (xy -4.122143 0.02) (xy -4.209286 -0.068571)
+				(xy -4.593571 -0.068571) (xy -4.707857 0.047143) (xy -4.707857 0.58) (xy -4.620714 0.667143) (xy -4.620714 0.781429)
+				(xy -4.665 0.781429)
+			)
+			(stroke
+				(width 0)
+				(type solid)
+			)
+			(fill yes)
+			(layer "F.SilkS")
+		)
+		(fp_poly
+			(pts
+				(xy 2.223571 1.071429) (xy 1.927857 0.777143) (xy 1.927857 -1.071429) (xy 2.332143 -1.071429) (xy 2.332143 -0.444286)
+				(xy 2.360714 -0.471429) (xy 3.026429 -0.471429) (xy 3.322143 -0.177143) (xy 3.322143 0.777143) (xy 3.026429 1.071429)
+				(xy 2.285 1.071429) (xy 2.285 0.964286) (xy 2.962143 0.964286) (xy 3.209286 0.717143) (xy 3.209286 -0.134286)
+				(xy 2.976429 -0.367143) (xy 2.379286 -0.367143) (xy 2.220714 -0.208571) (xy 2.220714 -0.964286)
+				(xy 2.037857 -0.964286) (xy 2.037857 0.717143) (xy 2.285 0.964286) (xy 2.285 1.071429) (xy 2.223571 1.071429)
+			)
+			(stroke
+				(width 0)
+				(type solid)
+			)
+			(fill yes)
+			(layer "F.SilkS")
+		)
+		(fp_poly
+			(pts
+				(xy -1.296429 1.071429) (xy -1.592143 0.777143) (xy -1.592143 -1.071429) (xy -1.187857 -1.071429)
+				(xy -1.187857 -0.444286) (xy -1.159286 -0.471429) (xy -0.493571 -0.471429) (xy -0.197857 -0.177143)
+				(xy -0.197857 0.777143) (xy -0.493571 1.071429) (xy -1.235 1.071429) (xy -1.235 0.964286) (xy -0.557857 0.964286)
+				(xy -0.310714 0.717143) (xy -0.310714 -0.134286) (xy -0.543571 -0.367143) (xy -1.140714 -0.367143)
+				(xy -1.299286 -0.208571) (xy -1.299286 -0.964286) (xy -1.482143 -0.964286) (xy -1.482143 0.717143)
+				(xy -1.235 0.964286) (xy -1.235 1.071429) (xy -1.296429 1.071429)
+			)
+			(stroke
+				(width 0)
+				(type solid)
+			)
+			(fill yes)
+			(layer "F.SilkS")
+		)
+		(fp_poly
+			(pts
+				(xy -4.816429 1.071429) (xy -5.112143 0.777143) (xy -5.112143 -1.071429) (xy -4.707857 -1.071429)
+				(xy -4.707857 -0.444286) (xy -4.679286 -0.471429) (xy -4.013571 -0.471429) (xy -3.717857 -0.177143)
+				(xy -3.717857 0.777143) (xy -4.013571 1.071429) (xy -4.755 1.071429) (xy -4.755 0.964286) (xy -4.077857 0.964286)
+				(xy -3.830714 0.717143) (xy -3.830714 -0.134286) (xy -4.063571 -0.367143) (xy -4.660714 -0.367143)
+				(xy -4.819286 -0.208571) (xy -4.819286 -0.964286) (xy -5.002143 -0.964286) (xy -5.002143 0.717143)
+				(xy -4.755 0.964286) (xy -4.755 1.071429) (xy -4.816429 1.071429)
+			)
+			(stroke
+				(width 0)
+				(type solid)
+			)
+			(fill yes)
+			(layer "F.SilkS")
+		)
+		(fp_poly
+			(pts
+				(xy 4.817857 -0.471429) (xy 5.112143 -0.177143) (xy 5.112143 0.23) (xy 4.817857 0.524286) (xy 4.040714 0.524286)
+				(xy 4.040714 0.58) (xy 4.127857 0.667143) (xy 5.092143 0.667143) (xy 5.092143 1.071429) (xy 3.979286 1.071429)
+				(xy 3.979286 0.962857) (xy 4.975 0.962857) (xy 4.975 0.78) (xy 4.069286 0.78) (xy 3.922143 0.632857)
+				(xy 3.922143 0.418571) (xy 4.767857 0.418571) (xy 5.000714 0.187143) (xy 5.000714 -0.121429) (xy 4.760714 -0.361429)
+				(xy 3.985 -0.361429) (xy 3.737857 -0.114286) (xy 3.737857 0.721429) (xy 3.979286 0.962857) (xy 3.979286 1.071429)
+				(xy 3.930714 1.071429) (xy 3.636429 0.777143) (xy 3.636429 -0.177143) (xy 3.930714 -0.471429) (xy 4.817857 -0.471429)
+			)
+			(stroke
+				(width 0)
+				(type solid)
+			)
+			(fill yes)
+			(layer "F.SilkS")
+		)
+		(fp_poly
+			(pts
+				(xy 1.297857 -0.471429) (xy 1.592143 -0.177143) (xy 1.592143 0.23) (xy 1.297857 0.524286) (xy 0.520714 0.524286)
+				(xy 0.520714 0.58) (xy 0.607857 0.667143) (xy 1.572143 0.667143) (xy 1.572143 1.071429) (xy 0.459286 1.071429)
+				(xy 0.459286 0.962857) (xy 1.455 0.962857) (xy 1.455 0.78) (xy 0.549286 0.78) (xy 0.402143 0.632857)
+				(xy 0.402143 0.418571) (xy 1.247857 0.418571) (xy 1.480714 0.187143) (xy 1.480714 -0.121429) (xy 1.240714 -0.361429)
+				(xy 0.465 -0.361429) (xy 0.217857 -0.114286) (xy 0.217857 0.721429) (xy 0.459286 0.962857) (xy 0.459286 1.071429)
+				(xy 0.410714 1.071429) (xy 0.116429 0.777143) (xy 0.116429 -0.177143) (xy 0.410714 -0.471429) (xy 1.297857 -0.471429)
+			)
+			(stroke
+				(width 0)
+				(type solid)
+			)
+			(fill yes)
+			(layer "F.SilkS")
+		)
+		(fp_poly
+			(pts
+				(xy -2.222143 -0.471429) (xy -1.927857 -0.177143) (xy -1.927857 0.23) (xy -2.222143 0.524286) (xy -2.999286 0.524286)
+				(xy -2.999286 0.58) (xy -2.912143 0.667143) (xy -1.947857 0.667143) (xy -1.947857 1.071429) (xy -3.060714 1.071429)
+				(xy -3.060714 0.962857) (xy -2.065 0.962857) (xy -2.065 0.78) (xy -2.970714 0.78) (xy -3.117857 0.632857)
+				(xy -3.117857 0.418571) (xy -2.272143 0.418571) (xy -2.039286 0.187143) (xy -2.039286 -0.121429)
+				(xy -2.279286 -0.361429) (xy -3.055 -0.361429) (xy -3.302143 -0.114286) (xy -3.302143 0.721429)
+				(xy -3.060714 0.962857) (xy -3.060714 1.071429) (xy -3.109286 1.071429) (xy -3.403571 0.777143)
+				(xy -3.403571 -0.177143) (xy -3.109286 -0.471429) (xy -2.222143 -0.471429)
+			)
+			(stroke
+				(width 0)
+				(type solid)
+			)
+			(fill yes)
+			(layer "F.SilkS")
+		)
+		(embedded_fonts no)
+	)
 	(footprint "Connector_PCBEdge:BUS_PCIexpress_x16"

Commit message: feat(gerbers): made order in jlcpcb and fixed document
Parts:
- removed kibuzzard-6911BE41: G***, kibuzzard-6911BE41
- added kibuzzard-691DF60A: G***, kibuzzard-691DF60A, F.Cu at (190.3, 50.0)
