File: schematics/alu_hub/alu_hub.kicad_sch (KiCad schematic)
At the start: 39 parts, among them U1 74LS574, U10 74LS02, U2 74LS245, U3 74LS02, U4 74LS181, U5 74LS181, U6 74LS574, U7 74LS245, U8 74LS245, U9 74LS02

Commit message: Push periphery and fix schematics
Connections:
- net HIGH4: now also U5.2 (A0); no longer U5.1 (B0)
- net HIGH5: now also U5.23 (A1); no longer U5.22 (B1)
- net HIGH6: now also U5.21 (A2); no longer U5.20 (B2)
- net HIGH7: now also U5.19 (A3); no longer U5.18 (B3)
- net LOW0: now also U4.1 (B0); no longer U5.2 (A0)
- net LOW1: now also U4.22 (B1); no longer U5.23 (A1)
- net LOW2: now also U4.20 (B2); no longer U5.21 (A2)
- net LOW3: now also U4.18 (B3); no longer U5.19 (A3)
- net LOW4: now also U5.1 (B0); no longer U4.1 (B0)
- net LOW5: now also U5.22 (B1); no longer U4.22 (B1)
- net LOW6: now also U5.20 (B2); no longer U4.20 (B2)
- net LOW7: now also U5.18 (B3); no longer U4.18 (B3)
Changed lines of the file:
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@@
 	)
 	(junction
+		(at 219.71 133.35)
+		(diameter 0)
+		(color 0 0 0 0)
+	)
+	(junction
 		(at 196.85 184.15)
 		(diameter 0)
@@
 	)
 	(junction
-		(at 240.03 100.33)
-		(diameter 0)
-		(color 0 0 0 0)
-	)
-	(junction
 		(at 86.36 59.69)
 		(diameter 0)
@@
 		)
 	)
-	(bus
-		(pts
-			(xy 205.74 125.73) (xy 240.03 125.73)
-		)
-		(stroke
-			(width 0)
-			(type default)
-		)
-	)
 	(wire
 		(pts
@@
 		)
 	)
-	(bus
+	(wire
 		(pts
-			(xy 240.03 100.33) (xy 243.84 100.33)
+			(xy 41.91 151.13) (xy 41.91 35.56)
 		)
 		(stroke
@@
 	(wire
 		(pts
-			(xy 41.91 151.13) (xy 41.91 35.56)
+			(xy 323.85 76.2) (xy 326.39 76.2)
 		)
 		(stroke
@@
 		)
 	)
-	(wire
+	(bus
 		(pts
-			(xy 323.85 76.2) (xy 326.39 76.2)
+			(xy 240.03 120.65) (xy 240.03 118.11)
 		)
 		(stroke
@@
 		)
 	)
-	(wire
+	(bus
 		(pts
-			(xy 142.24 147.32) (xy 142.24 173.99)
+			(xy 219.71 100.33) (xy 219.71 133.35)
 		)
 		(stroke
@@
 	(wire
 		(pts
-			(xy 191.77 195.58) (xy 191.77 218.44)
+			(xy 142.24 147.32) (xy 142.24 173.99)
 		)
 		(stroke
@@
 	(wire
 		(pts
-			(xy 270.51 195.58) (xy 270.51 190.5)
+			(xy 191.77 195.58) (xy 191.77 218.44)
 		)
 		(stroke
@@
 		)
 	)
-	(bus
+	(wire
 		(pts
-			(xy 240.03 120.65) (xy 240.03 123.19)
+			(xy 270.51 195.58) (xy 270.51 190.5)
 		)
 		(stroke
@@
 	(bus
 		(pts
-			(xy 240.03 128.27) (xy 240.03 130.81)
-		)
-		(stroke
-			(width 0)
-			(type default)
-		)
-	)
-	(bus
-		(pts
 			(xy 199.39 76.2) (xy 199.39 78.74)
 		)
@@
 		)
 	)
-	(bus
-		(pts
-			(xy 240.03 100.33) (xy 240.03 115.57)
-		)
-		(stroke
-			(width 0)
-			(type default)
-		)
-	)
 	(wire
 		(pts
@@
 		)
 	)
-	(bus
-		(pts
-			(xy 240.03 115.57) (xy 240.03 118.11)
-		)
-		(stroke
-			(width 0)
-			(type default)
-		)
-	)
 	(wire
 		(pts
@@
 	(bus
 		(pts
-			(xy 208.28 100.33) (xy 240.03 100.33)
+			(xy 207.01 133.35) (xy 219.71 133.35)
 		)
 		(stroke
@@
 		)
 	)
-	(bus
-		(pts
-			(xy 240.03 118.11) (xy 240.03 120.65)
-		)
-		(stroke
-			(width 0)
-			(type default)
-		)
-	)
 	(wire
 		(pts
@@
 	(bus
 		(pts
+			(xy 240.03 130.81) (xy 240.03 128.27)
+		)
+		(stroke
+			(width 0)
+			(type default)
+		)
+	)
+	(bus
+		(pts
 			(xy 86.36 76.2) (xy 86.36 78.74)
 		)
@@
 		)
 	)
+	(bus
+		(pts
+			(xy 205.74 115.57) (xy 240.03 115.57)
+		)
+		(stroke
+			(width 0)
+			(type default)
+		)
+	)
 	(wire
 		(pts
@@
 		)
 	)
+	(bus
+		(pts
+			(xy 219.71 100.33) (xy 243.84 100.33)
+		)
+		(stroke
+			(width 0)
+			(type default)
+		)
+	)
 	(wire
 		(pts
@@
 		)
 	)
+	(bus
+		(pts
+			(xy 240.03 120.65) (xy 240.03 123.19)
+		)
+		(stroke
+			(width 0)
+			(type default)
+		)
+	)
 	(wire
 		(pts
@@
 	(bus
 		(pts
-			(xy 205.74 100.33) (xy 205.74 125.73)
+			(xy 205.74 100.33) (xy 205.74 115.57)
 		)
 		(stroke
@@
 		)
 	)
+	(bus
+		(pts
+			(xy 240.03 133.35) (xy 240.03 130.81)
+		)
+		(stroke
+			(width 0)
+			(type default)
+		)
+	)
 	(wire
 		(pts
@@
 	(bus
 		(pts
-			(xy 208.28 100.33) (xy 208.28 180.34)
+			(xy 207.01 133.35) (xy 207.01 180.34)
 		)
 		(stroke
@@
 		)
 	)
-	(bus
-		(pts
-			(xy 240.03 130.81) (xy 240.03 133.35)
-		)
-		(stroke
-			(width 0)
-			(type default)
-		)
-	)
 	(wire
 		(pts
@@
 	(bus
 		(pts
-			(xy 208.28 180.34) (xy 134.62 180.34)
+			(xy 207.01 180.34) (xy 134.62 180.34)
 		)
 		(stroke
@@
 		)
 	)
+	(bus
+		(pts
+			(xy 219.71 133.35) (xy 240.03 133.35)
+		)
+		(stroke
+			(width 0)
+			(type default)
+		)
+	)
+	(bus
+		(pts
+			(xy 240.03 118.11) (xy 240.03 115.57)
+		)
+		(stroke
+			(width 0)
+			(type default)
+		)
+	)
 	(wire
 		(pts
@@
 		)
 	)
-	(label "HIGH5"
+	(label "LOW5"
 		(at 247.65 130.81 180)
 		(effects
@@
 		)
 	)
-	(label "LOW[0..7]"
-		(at 240.03 116.84 90)
-		(effects
-			(font
-				(size 1.27 1.27)
-			)
-			(justify left bottom)
-		)
-	)
 	(label "HIGH2"
 		(at 128.27 68.58 0)
@@
 		)
 	)
-	(label "HIGH4"
+	(label "LOW4"
 		(at 247.65 128.27 180)
 		(effects
@@
 		)
 	)
-	(label "LOW4"
+	(label "LOW0"
 		(at 143.51 124.46 180)
 		(effects
@@
 		)
 	)
-	(label "LOW6"
+	(label "LOW2"
 		(at 143.51 129.54 180)
 		(effects
@@
 		)
 	)
-	(label "LOW7"
+	(label "LOW3"
 		(at 143.51 132.08 180)
 		(effects
@@
 		)
 	)
-	(label "HIGH7"
+	(label "LOW7"
 		(at 247.65 135.89 180)
 		(effects
@@
 	)
 	(label "HIGH[0..7]"
-		(at 226.06 125.73 0)
+		(at 228.6 115.57 0)
 		(effects
 			(font
@@
 		)
 	)
-	(label "HIGH6"
+	(label "LOW6"
 		(at 247.65 133.35 180)
 		(effects
@@
 		)
 	)
-	(label "LOW1"
+	(label "HIGH5"
 		(at 247.65 120.65 180)
 		(effects
@@
 		)
 	)
-	(label "LOW3"
+	(label "LOW[0..7]"
+		(at 228.6 133.35 0)
+		(effects
+			(font
+				(size 1.27 1.27)
+			)
+			(justify left bottom)
+		)
+	)
+	(label "HIGH7"
 		(at 247.65 125.73 180)
 		(effects
@@
 		)
 	)
-	(label "LOW2"
+	(label "HIGH6"
 		(at 247.65 123.19 180)
 		(effects
@@
 		)
 	)
-	(label "LOW5"
+	(label "LOW1"
 		(at 143.51 127 180)
 		(effects
@@
 		)
 	)
-	(label "LOW0"
+	(label "HIGH4"
 		(at 247.65 118.11 180)
 		(effects
